Commit message: changes the urdf to be the real carlike one
Signed-off-by: Daniel Mascarenhas <daniel.mascarenhas@saipem.com>

File: urdf/carlike.urdf.xacro (robot description, xacro)
@@ -1,32 +1,214 @@
 <?xml version="1.0"?>
 <robot name="myfirst" xmlns:xacro="http://www.ros.org/wiki/xacro">
+<!--   <link name="base_link"> -->
+<!--     <visual> -->
+<!--       <origin xyz="0 0 0" rpy="0 0 0"/> -->
+<!--       <geometry> -->
+<!--         <box size="1 1 1"/> -->
+<!--       </geometry> -->
+<!--       <material name="red"> -->
+<!--         <color rgba="1 0 0 1"/> -->
+<!--       </material> -->
+<!--     </visual> -->
+<!--   </link> -->
+<!--   <link name="top_link"> -->
+<!--   <visual> -->
+<!--     <origin xyz="0 0 0" rpy="0 0 0"/> -->
+<!--     <geometry> -->
+<!--       <box size="0.5 0.5 0.5"/> -->
+<!--     </geometry> -->
+<!--     <material name="blue"> -->
+<!--       <color rgba="0 0 1 1"/> -->
+<!--     </material> -->
+<!--   </visual> -->
+<!-- </link> -->
+<!---->
+<!-- <joint name="base_to_top" type="revolute"> -->
+<!--   <parent link="base_link"/> -->
+<!--   <child link="top_link"/> -->
+<!--   <origin xyz="0 0 0.75" rpy="0 0 0"/> -->
+<!--   <limit lower="-1.57" upper="1.57" effort="10.0" velocity="1.0"/> -->
+<!--   <axis xyz="0 0 1"/> -->
+<!-- </joint> -->
+<!-- </robot> -->
+  <xacro:arg name="pkg" default="lar_car_like2"/>
+  <xacro:property name="mesh_dir" value="package://$(arg pkg)/urdf/meshes"/>
   <link name="base_link">
     <visual>
       <origin xyz="0 0 0" rpy="0 0 0"/>
       <geometry>
-        <box size="1 1 1"/>
-      </geometry>
-      <material name="red">
-        <color rgba="1 0 0 1"/>
-      </material>
-    </visual>
-  </link>
-  <link name="top_link">
-  <visual>
+        <mesh filename="${mesh_dir}/base_link.dae"/>
+      </geometry>
+    </visual>
+    <!-- <collision> -->
+    <!--   <origin xyz="0 0 0" rpy="0 0 0"/> -->
+    <!--   <geometry> -->
+    <!--     <box size="0.175621 0.225891 0.108579"/> -->
+    <!--   </geometry> -->
+    <!-- </collision> -->
+    <!-- <inertial> -->
+    <!--   <origin xyz="0 0 0" rpy="0 0 0"/> -->
+    <!--   <mass value="10.768651"/> -->
+    <!--   <inertia ixx="0.05637" ixy="0" ixz="0" iyy="0.038258" iyz="0" izz="0.073469"/> -->
+    <!-- </inertial> -->
+  </link>
+  <link name="front_left_steer_link">
+    <visual>
+      <origin xyz="0 0 0" rpy="0 0 0"/>
+      <geometry>
+        <mesh filename="${mesh_dir}/front_left_steer_link.dae"/>
+      </geometry>
+    </visual>
+    <!-- <collision> -->
+    <!--   <origin xyz="0 0 0" rpy="0 0 0"/> -->
+    <!--   <geometry> -->
+    <!--     <box size="0.033318 0.033356 0.003"/> -->
+    <!--   </geometry> -->
+    <!-- </collision> -->
+    <!-- <inertial> -->
+    <!--   <origin xyz="0 0 0" rpy="0 0 0"/> -->
+    <!--   <mass value="0.008335"/> -->
+    <!--   <inertia ixx="0.000001" ixy="0" ixz="0" iyy="0.000001" iyz="0" izz="0.000002"/> -->
+    <!-- </inertial> -->
+  </link>
+  <link name="front_right_steer_link">
+    <visual>
+      <origin xyz="0 0 0" rpy="0 0 0"/>
+      <geometry>
+        <mesh filename="${mesh_dir}/front_right_steer_link.dae"/>
+      </geometry>
+    </visual>
+    <!-- <collision> -->
+    <!--   <origin xyz="0 0 0" rpy="0 0 0"/> -->
+    <!--   <geometry> -->
+    <!--     <box size="0.033318 0.033356 0.003"/> -->
+    <!--   </geometry> -->
+    <!-- </collision> -->
+    <!-- <inertial> -->
+    <!--   <origin xyz="0 0 0" rpy="0 0 0"/> -->
+    <!--   <mass value="0.008335"/> -->
+    <!--   <inertia ixx="0.000001" ixy="0" ixz="0" iyy="0.000001" iyz="0" izz="0.000002"/> -->
+    <!-- </inertial> -->
+  </link>
+  <link name="front_left_wheel">
+    <visual>
+      <origin xyz="0 0 0" rpy="0 0 0"/>
+      <geometry>
+        <mesh filename="${mesh_dir}/front_left_wheel.dae"/>
+      </geometry>
+    </visual>
+    <!-- <collision> -->
+    <!--   <origin xyz="0 0 0" rpy="0 0 0"/> -->
+    <!--   <geometry> -->
+    <!--     <box size="31.650349 63 63"/> -->
+    <!--   </geometry> -->
+    <!-- </collision> -->
+    <!-- <inertial> -->
+    <!--   <origin xyz="0 0 0" rpy="0 0 0"/> -->
+    <!--   <mass value="314050584.611893"/> -->
+    <!--   <inertia ixx="207744461720.767029" ixy="0" ixz="0" iyy="130088769860.430832" iyz="0" izz="130088769860.430832"/> -->
+    <!-- </inertial> -->
+  </link>
+  <link name="front_right_wheel">
+    <visual>
+      <origin xyz="0 0 0" rpy="0 0 0"/>
+      <geometry>
+        <mesh filename="${mesh_dir}/front_right_wheel.dae"/>
+      </geometry>
+    </visual>
+    <!-- <collision> -->
+    <!--   <origin xyz="0 0 0" rpy="0 0 0"/> -->
+    <!--   <geometry> -->
+    <!--     <box size="31.500004 63 63"/> -->
+    <!--   </geometry> -->
+    <!-- </collision> -->
+    <!-- <inertial> -->
+    <!--   <origin xyz="0 0 0" rpy="0 0 0"/> -->
+    <!--   <mass value="312558787.851334"/> -->
+    <!--   <inertia ixx="206757638163.657196" ixy="0" ixz="0" iyy="129223530111.951172" iyz="0" izz="129223530111.951172"/> -->
+    <!-- </inertial> -->
+  </link>
+  <link name="rear_left_wheel">
+    <visual>
+      <origin xyz="0 0 0" rpy="0 0 0"/>
+      <geometry>
+        <mesh filename="${mesh_dir}/rear_left_wheel.dae"/>
+      </geometry>
+    </visual>
+    <!-- <collision> -->
+    <!--   <origin xyz="0 0 0" rpy="0 0 0"/> -->
+    <!--   <geometry> -->
+    <!--     <box size="31.500004 63 63.000008"/> -->
+    <!--   </geometry> -->
+    <!-- </collision> -->
+    <!-- <inertial> -->
+    <!--   <origin xyz="0 0 0" rpy="0 0 0"/> -->
+    <!--   <mass value="312558825.702672"/> -->
+    <!--   <inertia ixx="206757688240.982147" ixy="0" ixz="0" iyy="129223570799.779327" iyz="0" izz="129223545761.114563"/> -->
+    <!-- </inertial> -->
+  </link>
+  <link name="rear_right_wheel">
+    <visual>
+      <origin xyz="0 0 0" rpy="0 0 0"/>
+      <geometry>
+        <mesh filename="${mesh_dir}/rear_right_wheel.dae"/>
+      </geometry>
+    </visual>
+    <!-- <collision> -->
+    <!--   <origin xyz="0 0 0" rpy="0 0 0"/> -->
+    <!--   <geometry> -->
+    <!--     <box size="31.500004 63 63"/> -->
+    <!--   </geometry> -->
+    <!-- </collision> -->
+    <!-- <inertial> -->
+    <!--   <origin xyz="0 0 0" rpy="0 0 0"/> -->
+    <!--   <mass value="312558787.851334"/> -->
+    <!--   <inertia ixx="206757638163.657196" ixy="0" ixz="0" iyy="129223530111.951172" iyz="0" izz="129223530111.951172"/> -->
+    <!-- </inertial> -->
+  </link>
+  <!-- ========== JOINTS ========== -->
+  <joint name="front_left_steer_joint" type="revolute">
+    <parent link="base_link"/>
+    <child link="front_left_steer_link"/>
+    <origin xyz="-0.065239 0.066357 -0.017635" rpy="0 0 0"/>
+    <axis xyz="0 0 1"/>
+    <limit lower="-0.7" upper="0.7" effort="50" velocity="2.0"/>
+    <!-- <dynamics damping="1.0" friction="0.2"/> -->
+  </joint>
+  <joint name="front_right_steer_joint" type="revolute">
+    <parent link="base_link"/>
+    <child link="front_right_steer_link"/>
+    <origin xyz="0.072524 0.066228 -0.017635" rpy="0 0 0"/>
+    <axis xyz="0 0 1"/>
+    <limit lower="-0.7" upper="0.7" effort="50" velocity="2.0"/>
+    <!-- <dynamics damping="1.0" friction="0.2"/> -->
+  </joint>
+  <joint name="front_left_wheel_joint" type="continuous">
+    <parent link="front_left_steer_link"/>
+    <child link="front_left_wheel"/>
     <origin xyz="0 0 0" rpy="0 0 0"/>
-    <geometry>
-      <box size="0.5 0.5 0.5"/>
-    </geometry>
-    <material name="blue">
-      <color rgba="0 0 1 1"/>
-    </material>
-  </visual>
-</link>
-<joint name="base_to_top" type="revolute">
-  <parent link="base_link"/>
-  <child link="top_link"/>
-  <origin xyz="0 0 0.75" rpy="0 0 0"/>
-  <limit lower="-1.57" upper="1.57" effort="10.0" velocity="1.0"/>
-  <axis xyz="0 0 1"/>
-</joint>
+    <axis xyz="1 0 0"/>
+    <!-- <dynamics damping="0.1" friction="0.0"/> -->
+  </joint>
+  <joint name="front_right_wheel_joint" type="continuous">
+    <parent link="front_right_steer_link"/>
+    <child link="front_right_wheel"/>
+    <origin xyz="0 0 0" rpy="0 0 0"/>
+    <axis xyz="1 0 0"/>
+    <!-- <dynamics damping="0.1" friction="0.0"/> -->
+  </joint>
+  <joint name="rear_left_wheel_joint" type="continuous">
+    <parent link="base_link"/>
+    <child link="rear_left_wheel"/>
+    <origin xyz="-0.065282 -0.097208 -0.017635" rpy="0 0 0"/>
+    <axis xyz="1 0 0"/>
+    <dynamics damping="0.1" friction="0.0"/>
+  </joint>
+  <joint name="rear_right_wheel_joint" type="continuous">
+    <parent link="base_link"/>
+    <child link="rear_right_wheel"/>
+    <origin xyz="0.072523 -0.097281 -0.017635" rpy="0 0 0"/>
+    <axis xyz="1 0 0"/>
+    <!-- <dynamics damping="0.1" friction="0.0"/> -->
+  </joint>
 </robot>

File: urdf/carlike_minimal.urdf.xacro (robot description, xacro)
@@ -1,19 +1,32 @@
 <?xml version="1.0"?>
-<robot name="carlike">
-  <link name="world"/>
+<robot name="myfirst" xmlns:xacro="http://www.ros.org/wiki/xacro">
   <link name="base_link">
     <visual>
-      <origin xyz="0 0 0.3"/>
+      <origin xyz="0 0 0" rpy="0 0 0"/>
       <geometry>
-        <cylinder length="0.6" radius="0.2"/>
+        <box size="1 1 1"/>
       </geometry>
-      <material name="blue">
-        <color rgba="0 0 0.8 1"/>
+      <material name="red">
+        <color rgba="1 0 0 1"/>
       </material>
     </visual>
   </link>
-  <joint name="world_to_base" type="fixed">
-    <parent link="world"/>
-    <child link="base_link"/>
-  </joint>
+  <link name="top_link">
+  <visual>
+    <origin xyz="0 0 0" rpy="0 0 0"/>
+    <geometry>
+      <box size="0.5 0.5 0.5"/>
+    </geometry>
+    <material name="blue">
+      <color rgba="0 0 1 1"/>
+    </material>
+  </visual>
+</link>
+<joint name="base_to_top" type="revolute">
+  <parent link="base_link"/>
+  <child link="top_link"/>
+  <origin xyz="0 0 0.75" rpy="0 0 0"/>
+  <limit lower="-1.57" upper="1.57" effort="10.0" velocity="1.0"/>
+  <axis xyz="0 0 1"/>
+</joint>
 </robot>

Commit message: added basic control to the robot
Signed-off-by: Daniel Mascarenhas <daniel.mascarenhas@saipem.com>

File: urdf/carlike.urdf.xacro (robot description, xacro)
@@ -212,3 +212,38 @@
     <!-- <dynamics damping="0.1" friction="0.0"/> -->
   </joint>
+  <ros2_control name="CarLikeSystem" type="system">
+    <hardware>
+      <plugin>mock_components/GenericSystem</plugin>
+    </hardware>
+    <joint name="front_left_steer_joint">
+      <command_interface name="position"/>
+      <state_interface name="position"/>
+      <state_interface name="velocity"/>
+    </joint>
+    <joint name="front_right_steer_joint">
+      <command_interface name="position"/>
+      <state_interface name="position"/>
+      <state_interface name="velocity"/>
+    </joint>
+    <joint name="front_left_wheel_joint">
+      <command_interface name="velocity"/>
+      <state_interface name="position"/>
+      <state_interface name="velocity"/>
+    </joint>
+    <joint name="front_right_wheel_joint">
+      <command_interface name="velocity"/>
+      <state_interface name="position"/>
+      <state_interface name="velocity"/>
+    </joint>
+    <joint name="rear_left_wheel_joint">
+      <command_interface name="velocity"/>
+      <state_interface name="position"/>
+      <state_interface name="velocity"/>
+    </joint>
+    <joint name="rear_right_wheel_joint">
+      <command_interface name="velocity"/>
+      <state_interface name="position"/>
+      <state_interface name="velocity"/>
+    </joint>
+  </ros2_control>
 </robot>

Commit message: fixed axis of movement
Signed-off-by: Daniel Mascarenhas <daniel.mascarenhas@saipem.com>

File: urdf/carlike.urdf.xacro (robot description, xacro)
@@ -34,5 +34,8 @@
   <xacro:arg name="pkg" default="lar_car_like2"/>
   <xacro:property name="mesh_dir" value="package://$(arg pkg)/urdf/meshes"/>
-  <link name="base_link">
+  <!-- it seems that the vehicle has its front facing y instead of x -->
+  <!-- so I need to create a link to convert it -->
+  <link name="base_link"/>
+  <link name="chassis_link">
     <visual>
       <origin xyz="0 0 0" rpy="0 0 0"/>
@@ -95,5 +98,6 @@
       <origin xyz="0 0 0" rpy="0 0 0"/>
       <geometry>
-        <mesh filename="${mesh_dir}/front_left_wheel.dae"/>
+        <cylinder radius="0.0315" length="0.03"/>
+        <!-- <mesh filename="${mesh_dir}/front_left_wheel.dae"/> -->
       </geometry>
     </visual>
@@ -168,6 +172,11 @@
   </link>
   <!-- ========== JOINTS ========== -->
+  <joint name="base_link_to_chassis" type="fixed">
+    <parent link="base_link"/>
+    <child link="chassis_link"/>
+    <origin xyz="0 0 0" rpy="0 0 -1.57079632679"/>
+  </joint>
   <joint name="front_left_steer_joint" type="revolute">
-    <parent link="base_link"/>
+    <parent link="chassis_link"/>
     <child link="front_left_steer_link"/>
     <origin xyz="-0.065239 0.066357 -0.017635" rpy="0 0 0"/>
@@ -177,5 +186,5 @@
   </joint>
   <joint name="front_right_steer_joint" type="revolute">
-    <parent link="base_link"/>
+    <parent link="chassis_link"/>
     <child link="front_right_steer_link"/>
     <origin xyz="0.072524 0.066228 -0.017635" rpy="0 0 0"/>
@@ -199,5 +208,5 @@
   </joint>
   <joint name="rear_left_wheel_joint" type="continuous">
-    <parent link="base_link"/>
+    <parent link="chassis_link"/>
     <child link="rear_left_wheel"/>
     <origin xyz="-0.065282 -0.097208 -0.017635" rpy="0 0 0"/>
@@ -206,5 +215,5 @@
   </joint>
   <joint name="rear_right_wheel_joint" type="continuous">
-    <parent link="base_link"/>
+    <parent link="chassis_link"/>
     <child link="rear_right_wheel"/>
     <origin xyz="0.072523 -0.097281 -0.017635" rpy="0 0 0"/>
